File: hbridge/h-bridge.sch (EAGLE design)
At the start: 8 parts

Commit message: add connector parts
Parts:
- added R1, R2, R3, R4: (no value), resistor:R-US_R0603
- added U$2: JST-PH8-SMD-90, jst-ph:JST-PH8-SMD-90
Connections:
- new net N$2: R2.1, R3.1, R4.1, U$2.P$1
- net ENABLE: now also R1.2, U$2.P$8
- net GND: now also R1.1, R4.2
- net M1_DIR: now also U$2.P$6
- net M1_MOVE: now also U$2.P$7
- net M2_DIR: now also U$2.P$4
- net M2_MOVE: now also U$2.P$5
- net M3_DIR: now also U$2.P$2
- net M3_MOVE: now also U$2.P$3
- net V_RUN: now also R2.2, R3.2
Other:
- moved on the sheet: CONTROL
Changed lines of the file:
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@@
 <part name="GND6" library="supply1" deviceset="GND" device=""/>
 <part name="U$1" library="wolfbot" deviceset="ESWITCH-WSP1" device=""/>
+<part name="R1" library="resistor" deviceset="R-US_" device="R0603"/>
+<part name="U$2" library="jst-ph" deviceset="JST-PH8-SMD-90*" device=""/>
+<part name="R2" library="resistor" deviceset="R-US_" device="R0603"/>
+<part name="R3" library="resistor" deviceset="R-US_" device="R0603"/>
+<part name="R4" library="resistor" deviceset="R-US_" device="R0603"/>
+<part name="GND7" library="supply1" deviceset="GND" device=""/>
 </parts>
 <sheets>
@@
 <instance part="H2" gate="G$1" x="116.84" y="71.12"/>
 <instance part="MOTORS" gate="G$1" x="109.22" y="33.02" rot="MR180"/>
-<instance part="CONTROL" gate="G$1" x="55.88" y="33.02" rot="R180"/>
+<instance part="CONTROL" gate="G$1" x="86.36" y="33.02" rot="R180"/>
 <instance part="BAT" gate="G$1" x="53.34" y="109.22" rot="R180"/>
 <instance part="GND1" gate="1" x="83.82" y="68.58"/>
@@
 <instance part="GND6" gate="1" x="109.22" y="119.38"/>
 <instance part="U$1" gate="G$1" x="83.82" y="111.76"/>
+<instance part="R1" gate="G$1" x="-2.54" y="81.28" rot="R90"/>
+<instance part="U$2" gate="G$1" x="63.5" y="27.94" rot="MR180"/>
+<instance part="R2" gate="G$1" x="25.4" y="17.78" rot="R180"/>
+<instance part="R3" gate="G$1" x="25.4" y="17.78" rot="R180"/>
+<instance part="R4" gate="G$1" x="33.02" y="12.7" rot="R270"/>
+<instance part="GND7" gate="1" x="33.02" y="5.08"/>
 </instances>
 <busses>
@@
 <pinref part="H1" gate="G$1" pin="GND2"/>
 <wire x1="33.02" y1="68.58" x2="30.48" y2="68.58" width="0.1524" layer="91"/>
+<pinref part="R1" gate="G$1" pin="1"/>
+<wire x1="-2.54" y1="76.2" x2="-2.54" y2="73.66" width="0.1524" layer="91"/>
+<wire x1="-2.54" y1="73.66" x2="20.32" y2="73.66" width="0.1524" layer="91"/>
+<junction x="-2.54" y="76.2"/>
+<junction x="20.32" y="73.66"/>
 </segment>
 <segment>
@@
 <wire x1="114.3" y1="121.92" x2="109.22" y2="121.92" width="0.1524" layer="91"/>
 </segment>
+<segment>
+<pinref part="R4" gate="G$1" pin="2"/>
+<pinref part="GND7" gate="1" pin="GND"/>
+<junction x="33.02" y="7.62"/>
+</segment>
 </net>
 <net name="V+" class="1">
@@
 <segment>
 <pinref part="H1" gate="G$1" pin="1-2EN"/>
-<wire x1="33.02" y1="88.9" x2="22.86" y2="88.9" width="0.1524" layer="91"/>
-<label x="22.86" y="88.9" size="1.778" layer="95" rot="R180" xref="yes"/>
+<wire x1="33.02" y1="88.9" x2="-2.54" y2="88.9" width="0.1524" layer="91"/>
+<label x="-10.16" y="88.9" size="1.778" layer="95" rot="R180" xref="yes"/>
+<wire x1="-2.54" y1="88.9" x2="-10.16" y2="88.9" width="0.1524" layer="91"/>
+<wire x1="-2.54" y1="88.9" x2="-2.54" y2="86.36" width="0.1524" layer="91"/>
+<pinref part="R1" gate="G$1" pin="2"/>
+<junction x="-2.54" y="86.36"/>
 </segment>
 <segment>
@@
 </segment>
 <segment>
-<wire x1="50.8" y1="38.1" x2="45.72" y2="38.1" width="0.1524" layer="91"/>
+<wire x1="81.28" y1="38.1" x2="53.34" y2="38.1" width="0.1524" layer="91"/>
 <label x="45.72" y="38.1" size="1.778" layer="95" rot="R180" xref="yes"/>
 <pinref part="CONTROL" gate="G$1" pin="1"/>
+<pinref part="U$2" gate="G$1" pin="P$8"/>
+<wire x1="53.34" y1="38.1" x2="45.72" y2="38.1" width="0.1524" layer="91"/>
+<junction x="53.34" y="38.1"/>
 </segment>
 <segment>
@@
 </segment>
 <segment>
-<wire x1="50.8" y1="35.56" x2="30.48" y2="35.56" width="0.1524" layer="91"/>
+<wire x1="81.28" y1="35.56" x2="53.34" y2="35.56" width="0.1524" layer="91"/>
 <label x="30.48" y="35.56" size="1.778" layer="95" rot="R180" xref="yes"/>
 <pinref part="CONTROL" gate="G$1" pin="2"/>
+<pinref part="U$2" gate="G$1" pin="P$7"/>
+<wire x1="53.34" y1="35.56" x2="30.48" y2="35.56" width="0.1524" layer="91"/>
+<junction x="53.34" y="35.56"/>
 </segment>
 </net>
@@
 </segment>
 <segment>
-<wire x1="50.8" y1="33.02" x2="45.72" y2="33.02" width="0.1524" layer="91"/>
+<wire x1="81.28" y1="33.02" x2="53.34" y2="33.02" width="0.1524" layer="91"/>
 <label x="45.72" y="33.02" size="1.778" layer="95" rot="R180" xref="yes"/>
 <pinref part="CONTROL" gate="G$1" pin="3"/>
+<pinref part="U$2" gate="G$1" pin="P$6"/>
+<wire x1="53.34" y1="33.02" x2="45.72" y2="33.02" width="0.1524" layer="91"/>
+<junction x="53.34" y="33.02"/>
 </segment>
 </net>
@@
 </segment>
 <segment>
-<wire x1="50.8" y1="27.94" x2="45.72" y2="27.94" width="0.1524" layer="91"/>
+<wire x1="81.28" y1="27.94" x2="53.34" y2="27.94" width="0.1524" layer="91"/>
 <label x="45.72" y="27.94" size="1.778" layer="95" rot="R180" xref="yes"/>
 <pinref part="CONTROL" gate="G$1" pin="5"/>
+<pinref part="U$2" gate="G$1" pin="P$4"/>
+<wire x1="53.34" y1="27.94" x2="45.72" y2="27.94" width="0.1524" layer="91"/>
+<junction x="53.34" y="27.94"/>
 </segment>
 </net>
@@
 </segment>
 <segment>
-<wire x1="50.8" y1="30.48" x2="30.48" y2="30.48" width="0.1524" layer="91"/>
+<wire x1="81.28" y1="30.48" x2="53.34" y2="30.48" width="0.1524" layer="91"/>
 <label x="30.48" y="30.48" size="1.778" layer="95" rot="R180" xref="yes"/>
 <pinref part="CONTROL" gate="G$1" pin="4"/>
+<pinref part="U$2" gate="G$1" pin="P$5"/>
+<wire x1="53.34" y1="30.48" x2="30.48" y2="30.48" width="0.1524" layer="91"/>
+<junction x="53.34" y="30.48"/>
 </segment>
 </net>
@@
 </segment>
 <segment>
-<wire x1="50.8" y1="25.4" x2="30.48" y2="25.4" width="0.1524" layer="91"/>
+<wire x1="81.28" y1="25.4" x2="53.34" y2="25.4" width="0.1524" layer="91"/>
 <label x="30.48" y="25.4" size="1.778" layer="95" rot="R180" xref="yes"/>
 <pinref part="CONTROL" gate="G$1" pin="6"/>
+<pinref part="U$2" gate="G$1" pin="P$3"/>
+<wire x1="53.34" y1="25.4" x2="30.48" y2="25.4" width="0.1524" layer="91"/>
+<junction x="53.34" y="25.4"/>
 </segment>
 </net>
@@
 </segment>
 <segment>
-<wire x1="50.8" y1="22.86" x2="45.72" y2="22.86" width="0.1524" layer="91"/>
+<wire x1="81.28" y1="22.86" x2="53.34" y2="22.86" width="0.1524" layer="91"/>
 <label x="45.72" y="22.86" size="1.778" layer="95" rot="R180" xref="yes"/>
 <pinref part="CONTROL" gate="G$1" pin="7"/>
+<pinref part="U$2" gate="G$1" pin="P$2"/>
+<wire x1="53.34" y1="22.86" x2="45.72" y2="22.86" width="0.1524" layer="91"/>
+<junction x="53.34" y="22.86"/>
 </segment>
 </net>
@@
 <segment>
 <pinref part="H2" gate="G$1" pin="VCC1"/>
+<label x="137.16" y="88.9" size="1.778" layer="95" xref="yes"/>
 <wire x1="132.08" y1="88.9" x2="137.16" y2="88.9" width="0.1524" layer="91"/>
-<label x="137.16" y="88.9" size="1.778" layer="95" xref="yes"/>
+<label x="10.16" y="17.78" size="1.778" layer="95" rot="R180" xref="yes"/>
+<pinref part="R2" gate="G$1" pin="2"/>
+<pinref part="R3" gate="G$1" pin="2"/>
+<wire x1="10.16" y1="17.78" x2="20.32" y2="17.78" width="0.1524" layer="91"/>
+<junction x="20.32" y="17.78"/>
 </segment>
 <segment>
@@
 </segment>
 </net>
+<net name="N$2" class="0">
+<segment>
+<pinref part="R2" gate="G$1" pin="1"/>
+<pinref part="R3" gate="G$1" pin="1"/>
+<wire x1="30.48" y1="17.78" x2="33.02" y2="17.78" width="0.1524" layer="91"/>
+<pinref part="U$2" gate="G$1" pin="P$1"/>
+<wire x1="33.02" y1="17.78" x2="45.72" y2="17.78" width="0.1524" layer="91"/>
+<wire x1="45.72" y1="17.78" x2="45.72" y2="20.32" width="0.1524" layer="91"/>
+<wire x1="45.72" y1="20.32" x2="53.34" y2="20.32" width="0.1524" layer="91"/>
+<junction x="53.34" y="20.32"/>
+<junction x="30.48" y="17.78"/>
+<pinref part="R4" gate="G$1" pin="1"/>
+<junction x="33.02" y="17.78"/>
+</segment>
+</net>

Commit message: tested and fixed until passed Sparkfun's DRC
Parts:
- removed CONTROL: (no value), SparkFun-Connectors:M07LOCK
- removed R2, R3: (no value), resistor:R-US_R0603
- removed U$2: JST-PH8-SMD-90, jst-ph:JST-PH8-SMD-90
- added BATT_H: (no value), resistor:R-US_R0603
- added U$3: JST-PH8-SMD-90, jst-ph:JST-PH8-SMD-90
- renumbered R4 to BATT_L
Connections:
- net ENABLE: now also U$3.P$1; no longer CONTROL.1, U$2.P$8
- net M1_DIR: now also U$3.P$3; no longer CONTROL.3, U$2.P$6
- net M1_MOVE: now also U$3.P$2; no longer CONTROL.2, U$2.P$7
- net M2_DIR: now also U$3.P$5; no longer CONTROL.5, U$2.P$4
- net M2_MOVE: now also U$3.P$4; no longer CONTROL.4, U$2.P$5
- net M3_DIR: now also U$3.P$7; no longer CONTROL.7, U$2.P$2
- net M3_MOVE: now also U$3.P$6; no longer CONTROL.6, U$2.P$3
- net N$2: now also BATT_H.1, U$3.P$8; no longer R2.1, R3.1, U$2.P$1
- net V_RUN: now also BATT_H.2; no longer R2.2, R3.2
Changed lines of the file:
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@@
 <part name="H2" library="st-microelectronics" deviceset="L293D" device=""/>
 <part name="MOTORS" library="SparkFun-Connectors" deviceset="M06" device="LOCK"/>
-<part name="CONTROL" library="SparkFun-Connectors" deviceset="M07" device="LOCK"/>
 <part name="BAT" library="con-molex-micro-fit-3_0" deviceset="HEADER_POS2_?" device="43045-0206"/>
 <part name="GND1" library="supply1" deviceset="GND" device=""/>
@@
 <part name="U$1" library="wolfbot" deviceset="ESWITCH-WSP1" device=""/>
 <part name="R1" library="resistor" deviceset="R-US_" device="R0603"/>
-<part name="U$2" library="jst-ph" deviceset="JST-PH8-SMD-90*" device=""/>
-<part name="R2" library="resistor" deviceset="R-US_" device="R0603"/>
-<part name="R3" library="resistor" deviceset="R-US_" device="R0603"/>
-<part name="R4" library="resistor" deviceset="R-US_" device="R0603"/>
+<part name="BATT_H" library="resistor" deviceset="R-US_" device="R0603"/>
+<part name="BATT_L" library="resistor" deviceset="R-US_" device="R0603"/>
 <part name="GND7" library="supply1" deviceset="GND" device=""/>
+<part name="U$3" library="jst-ph" deviceset="JST-PH8-SMD-90*" device=""/>
 </parts>
 <sheets>
@@
 <instance part="H2" gate="G$1" x="116.84" y="71.12"/>
 <instance part="MOTORS" gate="G$1" x="109.22" y="33.02" rot="MR180"/>
-<instance part="CONTROL" gate="G$1" x="86.36" y="33.02" rot="R180"/>
 <instance part="BAT" gate="G$1" x="53.34" y="109.22" rot="R180"/>
 <instance part="GND1" gate="1" x="83.82" y="68.58"/>
@@
 <instance part="U$1" gate="G$1" x="83.82" y="111.76"/>
 <instance part="R1" gate="G$1" x="-2.54" y="81.28" rot="R90"/>
-<instance part="U$2" gate="G$1" x="63.5" y="27.94" rot="MR180"/>
-<instance part="R2" gate="G$1" x="25.4" y="17.78" rot="R180"/>
-<instance part="R3" gate="G$1" x="25.4" y="17.78" rot="R180"/>
-<instance part="R4" gate="G$1" x="33.02" y="12.7" rot="R270"/>
+<instance part="BATT_H" gate="G$1" x="22.86" y="17.78" rot="R180"/>
+<instance part="BATT_L" gate="G$1" x="33.02" y="12.7" rot="R270"/>
 <instance part="GND7" gate="1" x="33.02" y="5.08"/>
+<instance part="U$3" gate="G$1" x="60.96" y="30.48"/>
 </instances>
 <busses>
@@
 </segment>
 <segment>
-<pinref part="R4" gate="G$1" pin="2"/>
+<pinref part="BATT_L" gate="G$1" pin="2"/>
 <pinref part="GND7" gate="1" pin="GND"/>
 <junction x="33.02" y="7.62"/>
@@
 <pinref part="R1" gate="G$1" pin="2"/>
 <junction x="-2.54" y="86.36"/>
+<junction x="-2.54" y="88.9"/>
 </segment>
 <segment>
@@
 </segment>
 <segment>
-<wire x1="81.28" y1="38.1" x2="53.34" y2="38.1" width="0.1524" layer="91"/>
 <label x="45.72" y="38.1" size="1.778" layer="95" rot="R180" xref="yes"/>
-<pinref part="CONTROL" gate="G$1" pin="1"/>
-<pinref part="U$2" gate="G$1" pin="P$8"/>
-<wire x1="53.34" y1="38.1" x2="45.72" y2="38.1" width="0.1524" layer="91"/>
-<junction x="53.34" y="38.1"/>
+<pinref part="U$3" gate="G$1" pin="P$1"/>
+<wire x1="50.8" y1="38.1" x2="45.72" y2="38.1" width="0.1524" layer="91"/>
 </segment>
 <segment>
@@
 </segment>
 <segment>
-<wire x1="81.28" y1="35.56" x2="53.34" y2="35.56" width="0.1524" layer="91"/>
 <label x="30.48" y="35.56" size="1.778" layer="95" rot="R180" xref="yes"/>
-<pinref part="CONTROL" gate="G$1" pin="2"/>
-<pinref part="U$2" gate="G$1" pin="P$7"/>
-<wire x1="53.34" y1="35.56" x2="30.48" y2="35.56" width="0.1524" layer="91"/>
-<junction x="53.34" y="35.56"/>
+<pinref part="U$3" gate="G$1" pin="P$2"/>
+<wire x1="50.8" y1="35.56" x2="30.48" y2="35.56" width="0.1524" layer="91"/>
 </segment>
 </net>
@@
 </segment>
 <segment>
-<wire x1="81.28" y1="33.02" x2="53.34" y2="33.02" width="0.1524" layer="91"/>
 <label x="45.72" y="33.02" size="1.778" layer="95" rot="R180" xref="yes"/>
-<pinref part="CONTROL" gate="G$1" pin="3"/>
-<pinref part="U$2" gate="G$1" pin="P$6"/>
-<wire x1="53.34" y1="33.02" x2="45.72" y2="33.02" width="0.1524" layer="91"/>
-<junction x="53.34" y="33.02"/>
+<pinref part="U$3" gate="G$1" pin="P$3"/>
+<wire x1="50.8" y1="33.02" x2="45.72" y2="33.02" width="0.1524" layer="91"/>
 </segment>
 </net>
@@
 </segment>
 <segment>
-<wire x1="81.28" y1="27.94" x2="53.34" y2="27.94" width="0.1524" layer="91"/>
 <label x="45.72" y="27.94" size="1.778" layer="95" rot="R180" xref="yes"/>
-<pinref part="CONTROL" gate="G$1" pin="5"/>
-<pinref part="U$2" gate="G$1" pin="P$4"/>
-<wire x1="53.34" y1="27.94" x2="45.72" y2="27.94" width="0.1524" layer="91"/>
-<junction x="53.34" y="27.94"/>
+<pinref part="U$3" gate="G$1" pin="P$5"/>
+<wire x1="50.8" y1="27.94" x2="45.72" y2="27.94" width="0.1524" layer="91"/>
 </segment>
 </net>
@@
 </segment>
 <segment>
-<wire x1="81.28" y1="30.48" x2="53.34" y2="30.48" width="0.1524" layer="91"/>
 <label x="30.48" y="30.48" size="1.778" layer="95" rot="R180" xref="yes"/>
-<pinref part="CONTROL" gate="G$1" pin="4"/>
-<pinref part="U$2" gate="G$1" pin="P$5"/>
-<wire x1="53.34" y1="30.48" x2="30.48" y2="30.48" width="0.1524" layer="91"/>
-<junction x="53.34" y="30.48"/>
+<pinref part="U$3" gate="G$1" pin="P$4"/>
+<wire x1="50.8" y1="30.48" x2="30.48" y2="30.48" width="0.1524" layer="91"/>
 </segment>
 </net>
@@
 </segment>
 <segment>
-<wire x1="81.28" y1="25.4" x2="53.34" y2="25.4" width="0.1524" layer="91"/>
 <label x="30.48" y="25.4" size="1.778" layer="95" rot="R180" xref="yes"/>
-<pinref part="CONTROL" gate="G$1" pin="6"/>
-<pinref part="U$2" gate="G$1" pin="P$3"/>
-<wire x1="53.34" y1="25.4" x2="30.48" y2="25.4" width="0.1524" layer="91"/>
-<junction x="53.34" y="25.4"/>
+<pinref part="U$3" gate="G$1" pin="P$6"/>
+<wire x1="50.8" y1="25.4" x2="30.48" y2="25.4" width="0.1524" layer="91"/>
 </segment>
 </net>
@@
 </segment>
 <segment>
-<wire x1="81.28" y1="22.86" x2="53.34" y2="22.86" width="0.1524" layer="91"/>
 <label x="45.72" y="22.86" size="1.778" layer="95" rot="R180" xref="yes"/>
-<pinref part="CONTROL" gate="G$1" pin="7"/>
-<pinref part="U$2" gate="G$1" pin="P$2"/>
-<wire x1="53.34" y1="22.86" x2="45.72" y2="22.86" width="0.1524" layer="91"/>
-<junction x="53.34" y="22.86"/>
+<pinref part="U$3" gate="G$1" pin="P$7"/>
+<wire x1="50.8" y1="22.86" x2="45.72" y2="22.86" width="0.1524" layer="91"/>
 </segment>
 </net>
@@
 </segment>
 <segment>
-<pinref part="H2" gate="G$1" pin="VCC1"/>
-<label x="137.16" y="88.9" size="1.778" layer="95" xref="yes"/>
-<wire x1="132.08" y1="88.9" x2="137.16" y2="88.9" width="0.1524" layer="91"/>
 <label x="10.16" y="17.78" size="1.778" layer="95" rot="R180" xref="yes"/>
-<pinref part="R2" gate="G$1" pin="2"/>
-<pinref part="R3" gate="G$1" pin="2"/>
-<wire x1="10.16" y1="17.78" x2="20.32" y2="17.78" width="0.1524" layer="91"/>
-<junction x="20.32" y="17.78"/>
+<pinref part="BATT_H" gate="G$1" pin="2"/>
+<wire x1="10.16" y1="17.78" x2="17.78" y2="17.78" width="0.1524" layer="91"/>
 </segment>
 <segment>
@@
 <wire x1="33.02" y1="53.34" x2="22.86" y2="53.34" width="0.1524" layer="91"/>
 <label x="22.86" y="53.34" size="1.778" layer="95" rot="R180" xref="yes"/>
+</segment>
+<segment>
+<pinref part="H2" gate="G$1" pin="VCC1"/>
+<wire x1="132.08" y1="88.9" x2="137.16" y2="88.9" width="0.1524" layer="91"/>
+<label x="137.16" y="88.9" size="1.778" layer="95" xref="yes"/>
 </segment>
 </net>
@@
 <net name="N$2" class="0">
 <segment>
-<pinref part="R2" gate="G$1" pin="1"/>
-<pinref part="R3" gate="G$1" pin="1"/>
-<wire x1="30.48" y1="17.78" x2="33.02" y2="17.78" width="0.1524" layer="91"/>
-<pinref part="U$2" gate="G$1" pin="P$1"/>
+<pinref part="BATT_H" gate="G$1" pin="1"/>
+<wire x1="27.94" y1="17.78" x2="33.02" y2="17.78" width="0.1524" layer="91"/>
 <wire x1="33.02" y1="17.78" x2="45.72" y2="17.78" width="0.1524" layer="91"/>
 <wire x1="45.72" y1="17.78" x2="45.72" y2="20.32" width="0.1524" layer="91"/>
-<wire x1="45.72" y1="20.32" x2="53.34" y2="20.32" width="0.1524" layer="91"/>
-<junction x="53.34" y="20.32"/>
-<junction x="30.48" y="17.78"/>
-<pinref part="R4" gate="G$1" pin="1"/>
+<wire x1="45.72" y1="20.32" x2="50.8" y2="20.32" width="0.1524" layer="91"/>
+<pinref part="BATT_L" gate="G$1" pin="1"/>
 <junction x="33.02" y="17.78"/>
-</segment>
-</net>
+<pinref part="U$3" gate="G$1" pin="P$8"/>
+</segment>
+</net>
