File: boards/power/powerboard.brd (EAGLE design)
At the start: 83 x 42 mm, 55 parts, among them IC1 TPS5420, IC2 TPS5420

Commit message: Changing boards for fet and text improvements
Parts:
- R2, R4: value (none) -> 500
Changed lines of the file:
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@@
 <attribute name="VALUE" x="34.1432" y="33.6304" size="1.27" layer="27"/>
 </element>
-<element name="R2" library="rcl" package="R3216" value="" x="4.6482" y="8.636" smashed="yes" rot="R180">
+<element name="R2" library="rcl" package="R3216" value="500" x="4.6482" y="8.636" smashed="yes" rot="R180">
 <attribute name="NAME" x="0.9144" y="9.0678" size="0.6096" layer="25" rot="R270"/>
 <attribute name="VALUE" x="6.5532" y="11.176" size="1.27" layer="27" rot="R180"/>
 </element>
-<element name="R4" library="rcl" package="R3216" value="" x="32.3342" y="37.0078" smashed="yes" rot="R90">
+<element name="R4" library="rcl" package="R3216" value="500" x="32.3342" y="37.0078" smashed="yes" rot="R90">
 <attribute name="NAME" x="30.988" y="36.4998" size="0.6096" layer="25" rot="R90"/>
 <attribute name="VALUE" x="34.8742" y="35.1028" size="1.27" layer="27" rot="R90"/>

Commit message: New board for plugin regulator
Parts:
- removed CBP: 100nF, rcl:C0805
- removed CCOMP: 120nF, rcl:C0805
- removed CCOMP2: 510pF, rcl:C0805
- removed CIN: 22uF, rcl:C0805
- removed COUT, COUT1: 56uF, rcl:SANYO-OSCON_SMD_A5
- removed CRAMP: 750pF, rcl:C0805
- removed CSEP: 2.2uF, rcl:C0805
- removed LIN: 6.2uH, SparkFun-Passives:SRU1038
- removed LOUT: 15uH, SparkFun-Passives:SRU1038
- removed RBP: 20.0, rcl:R0805
- removed RCOMP: 1.47k, rcl:R0805
- removed RFADJ: 34.8k, rcl:R0805
- removed RFB1: 10k, rcl:R0805
- removed RFB2: 37.4k, rcl:R0805
- removed RRAMP: 100.0, rcl:R0805
- removed RSENSE: 0.016, rcl:R2512
- removed U$5: P-CHANNEL20V(D-S)MOSFET, ngohara_parts:TSOP-6
- removed U$6: DPAK_DIODE, ngohara_parts:DPAK
- added JP1: (no value), SparkFun-Connectors:1X04_LOCK
- added R10, R11, R8, R9: 0, resistor:R0805
- added U$4: THERMAL_PAD, ngohara_parts:THERMAL_PAD
- U$2: value LM3488 -> THERMAL_PAD; device 40xx:SO08 -> ngohara_parts:THERMAL_PAD
- moved U$2 27.2 mm to (75.9, 34.0), turned to 0 degrees
- moved X3 3.30 mm to (80.6, 4.90), turned to 90 degrees
- moved U$1 2.27 mm to (50.3, 33.4)
Connections:
- removed net 6V: COUT.+, COUT1.+, RFB2.1, U$6.4, X3.P$2
- removed net FB: RFB1.1, RFB2.2, U$2.3
- removed net LINSIG: CSEP.1, LIN.2, U$5.P$4
- removed net LSIG: CSEP.2, LOUT.1, U$6.1, U$6.3
- removed net N$1: CCOMP.1, RCOMP.1
- removed net N$20: RFADJ.2, U$2.7
- removed net N$21: CRAMP.1, RRAMP.2, U$2.1
- removed net N$23: U$2.6, U$5.P$3
- removed net N$3: CCOMP2.1, RCOMP.2, U$2.2
- removed net N$9: CBP.1, RBP.1, U$2.8
- removed net SIG1: RRAMP.1, RSENSE.2, U$5.P$1, U$5.P$2, U$5.P$5, U$5.P$6
- new net 6VOUT: JP1.4, X3.P$2
- new net VIN: JP1.2, R10.2, R11.2, R8.2, R9.2
- net 5V: now also R10.1, R11.1
- net GND: now also JP1.3; no longer CBP.2, CCOMP.2, CCOMP2.2, CIN.2, COUT.-, COUT1.-, CRAMP.2, LOUT.2, RFADJ.1, RFB1.2, RSENSE.1, U$2.4, U$2.5
- net V_BATT: now also R8.1, R9.1; no longer CIN.1, LIN.1, RBP.2
Routing:
- net FB: track 39.3 -> 0.00 mm, vias 2 -> 0
- net 6VOUT: track 0.00 -> 37.5 mm, vias 0 -> 1
- net N$9: track 30.0 -> 0.00 mm, vias 2 -> 0
- net VIN: track 0.00 -> 26.9 mm, vias 0 -> 1
- net N$3: track 25.2 -> 0.00 mm, vias 2 -> 0
- net N$21: track 24.1 -> 0.00 mm, vias 2 -> 0
- net 5V: track 0.00 -> 23.2 mm
- net N$23: track 19.4 -> 0.00 mm, vias 2 -> 0
- net GND: track 19.1 -> 0.37 mm, vias 6 -> 3
- net N$20: track 10.4 -> 0.00 mm, vias 2 -> 0
- net N$6: track 22.4 -> 27.2 mm
- net V_BATT: track 73.6 -> 69.7 mm
- net N$1: track 2.79 -> 0.00 mm
- added copper zone on layer 1, net VIN
- removed copper zone on layer 1, net 6V
- removed copper zone on layer 1, net LINSIG
- removed copper zone on layer 1, net LSIG
- removed copper zone on layer 1, net SIG1
Other:
- board text added: "5V short"
- board text added: "BATT. short"
- board text removed: "."
- board text removed: "1"
