File: boards/power/powerboard.brd (EAGLE design)
At the start: 83 x 42 mm, 42 parts, among them IC1 TPS5420, IC2 TPS5420

Commit message: Cleanup issues, working on powerboard res move
Routing:
- net GND: vias 3 -> 5
Other:
- board text added: "v.2013/09/26"
- board text removed: "REV. Aug 8 2013"
Changed lines of the file:
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@@
 <text x="17.2938" y="28.7532" size="1.27" layer="26" font="vector" ratio="11" rot="MR180">7.4V= 3.3V, 5V,  6V @ 2A MAX</text>
 <text x="24.1264" y="25.7052" size="1.016" layer="26" font="vector" ratio="16" rot="MR180">Wolfbot Swarm Robotics</text>
-<text x="26.3362" y="23.7494" size="1.016" layer="26" font="vector" ratio="16" rot="MR180">REV. Aug 8 2013</text>
+<text x="26.3362" y="23.7494" size="1.016" layer="26" font="vector" ratio="16" rot="MR180">v.2013/09/26</text>
 <text x="60.452" y="20.066" size="1.016" layer="25" font="vector" rot="R90">5V short</text>
 <text x="60.706" y="8.89" size="1.016" layer="25" font="vector" rot="R90">BATT. short</text>
@@
 <contactref element="X2" pad="P$1"/>
 <polygon width="0.508" layer="1" spacing="1.016" isolate="0.8128">
-<vertex x="19.0246" y="34.2138"/>
-<vertex x="11.43" y="34.1884"/>
-<vertex x="11.4046" y="37.592"/>
+<vertex x="19.0246" y="34.29"/>
+<vertex x="0.762" y="34.29"/>
+<vertex x="0.762" y="41.148"/>
+<vertex x="12.954" y="41.148"/>
+<vertex x="12.954" y="37.592"/>
 <vertex x="33.1132" y="37.592"/>
 <vertex x="33.1894" y="35.2044"/>
@@
 <via x="59.5568" y="5.3414" extent="1-16" drill="0.6" alwaysstop="yes"/>
 <contactref element="C19" pad="2"/>
+<via x="3.8246" y="4" extent="1-16" drill="3.2" diameter="5.5" alwaysstop="yes"/>
+<via x="3.8246" y="38" extent="1-16" drill="3.2" diameter="5.5" alwaysstop="yes"/>
 </signal>
 <signal name="N$6">
@@
 <via x="65.8246" y="4" extent="1-16" drill="3.2" diameter="5.5" alwaysstop="yes"/>
 </signal>
-<signal name="N$15">
-<via x="3.8246" y="4" extent="1-16" drill="3.2" diameter="5.5" alwaysstop="yes"/>
-</signal>
-<signal name="N$16">
-<via x="3.8246" y="38" extent="1-16" drill="3.2" diameter="5.5" alwaysstop="yes"/>
-</signal>
 <signal name="N$17">
