File: boards/usb/usb.sch (EAGLE design)
At the start: 3 parts

Commit message: Minor tweaks to USB board: wider, silkscreen
- wider so male USB can be moved in for better support
- added version stamp and tweaked other silk
- labeled signal lines in schematic
- added dimension layer to top silk in CAM job
Connections:
- net N$3 renamed D+
- net N$4 renamed D-
Changed lines of the file:
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@@
 <setting verticaltext="up"/>
 </settings>
-<grid distance="0.01" unitdist="inch" unit="inch" style="lines" multiple="1" display="no" altdistance="0.01" altunitdist="inch" altunit="inch"/>
+<grid distance="0.1" unitdist="inch" unit="inch" style="lines" multiple="1" display="no" altdistance="0.01" altunitdist="inch" altunit="inch"/>
 <layers>
 <layer number="1" name="Top" color="4" fill="1" visible="no" active="no"/>
@@
 </busses>
 <nets>
-<net name="N$3" class="0">
+<net name="D+" class="0">
 <segment>
 <pinref part="U$1" gate="G$1" pin="D+"/>
@@
 </segment>
 </net>
-<net name="N$4" class="0">
+<net name="D-" class="0">
 <segment>
 <pinref part="U$2" gate="G$1" pin="D-"/>
